Commit message: 修改驱动轮碰撞体积

File: resources/robots/wl/urdf/wl.urdf (robot description, URDF)
Before this commit: robot wl, 7 links, 6 joints
Links:
- link l_Wheel_Link: geometry collision cylinder length=0.025 radius=0.0675; visual mesh filename=../meshes/l_Wheel_Link.dae
- link r_Wheel_Link: geometry collision cylinder length=0.025 radius=0.0675; visual mesh filename=../meshes/r_Wheel_Link.dae
