Commit message: add cubli

File: resources/robots/cubli/urdf/cubli.urdf (robot description, URDF)
Before this commit: robot cubli, 4 links, 3 joints
Links:
- link base: geometry collision mesh filename=../meshes/base.dae; visual mesh filename=../meshes/base.dae
- link wheel1: geometry collision mesh filename=../meshes/wheel1.dae; visual mesh filename=../meshes/wheel1.dae
- link wheel2: geometry collision mesh filename=../meshes/wheel2.dae; visual mesh filename=../meshes/wheel2.dae
- link wheel3: geometry collision mesh filename=../meshes/wheel3.dae; visual mesh filename=../meshes/wheel3.dae
