Commit message: add nezha

File: resources/robots/nezha2/urdf/nezha2.urdf (robot description, URDF)
Before this commit: robot nezha2, 17 links, 16 joints
Links:
- removed link hip_left_bar_link
- removed link hip_left_crank_link
- removed link hip_right_bar_link
- removed link hip_right_crank_lin
- removed link knee_left_bar_link
- removed link knee_left_crank_link
- removed link knee_right_bar_link
- removed link knee_right_crank_link
- link body_link: geometry collision mesh filename=../meshes/body_link.STL; visual mesh filename=../meshes/body_link.STL
- link passiveWheel_left_link: geometry collision mesh filename=../meshes/passiveWheel_left_link.STL; visual mesh filename=../meshes/passiveWheel_left_link.STL
- link passiveWheel_right_link: geometry collision mesh filename=../meshes/passiveWheel_right_link.STL; visual mesh filename=../meshes/passiveWheel_right_link.STL
- link shank_left_link: geometry collision mesh filename=../meshes/shank_left_link.STL; visual mesh filename=../meshes/shank_left_link.STL
- link shank_right_link: geometry collision mesh filename=../meshes/shank_right_link.STL; visual mesh filename=../meshes/shank_right_link.STL
- link thigh_left_link: geometry collision mesh filename=../meshes/thigh_left_link.STL; visual mesh filename=../meshes/thigh_left_link.STL
- link thigh_right_link: geometry collision mesh filename=../meshes/thigh_right_link.STL; visual mesh filename=../meshes/thigh_right_link.STL
- link wheel_left_link: geometry collision mesh filename=../meshes/wheel_left_link.STL; visual mesh filename=../meshes/wheel_left_link.STL
- link wheel_right_link: geometry collision mesh filename=../meshes/wheel_right_link.STL; visual mesh filename=../meshes/wheel_right_link.STL
Joints:
- removed joint hip_left_bar_joint
- removed joint hip_left_motor_joint
- removed joint hip_right_bar_joint
- removed joint hip_right_motor_joint
- removed joint knee_left_bar_joint
- removed joint knee_left_motor_joint
- removed joint knee_right_bar_joint
- removed joint knee_right_motor_joint
